File: jduino.sch (EAGLE design)
At the start: 18 parts, among them IC1 LM2936Z-5.0, IC2 ATMEGA48/88/168-PU, J1 Analog I/O, J2 Digital I/O, J3 Digital I/O, J5 Power Jumpers, J6 FTDI Jumpers, Q1 16 mHz

Commit message: Initial attempt at hand routing.
The ATmega needs to be moved to the left to allow enough space to
route all of the digital I/O pins.
Parts:
- removed J7: (no value), con-jack:JACK-PLUG1
- added J4: POWER_JACKPTH, SparkFun-Connectors:POWER_JACKPTH
- added LED2: LED13, led:LED3MM
- added R3: 330, rcl:R-US_0204/5
- IC1: value LM2936Z-5.0 -> LM2937-5.0; device national-semiconductor:LM2936Z-5.0 -> SparkFun-PowerIC:V_REG_78XX-TO-220
Connections:
- new net N$4: LED2.C, R3.2
- net +5V: now also IC1.OUT; no longer IC1.VO
- net D13: now also LED2.A
- net GND: now also J4.GNDBREAK, R3.1; no longer J7.1, J7.2
- net N$2: now also J4.PWR; no longer J7.3
- net N$6: now also IC1.IN; no longer IC1.VIN
Changed lines of the file:
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@@
 <layer number="106" name="bPlate" color="7" fill="1" visible="yes" active="yes"/>
 <layer number="107" name="Crop" color="7" fill="1" visible="yes" active="yes"/>
+<layer number="108" name="tplace-old" color="10" fill="1" visible="yes" active="yes"/>
+<layer number="109" name="ref-old" color="11" fill="1" visible="yes" active="yes"/>
 <layer number="116" name="Patch_BOT" color="9" fill="4" visible="yes" active="yes"/>
 <layer number="121" name="_tsilk" color="7" fill="1" visible="yes" active="yes"/>
@@
 <layer number="144" name="Drill_legend" color="7" fill="1" visible="no" active="yes"/>
 <layer number="151" name="HeatSink" color="7" fill="1" visible="yes" active="yes"/>
+<layer number="199" name="Contour" color="7" fill="1" visible="yes" active="yes"/>
 <layer number="200" name="200bmp" color="1" fill="10" visible="yes" active="yes"/>
 <layer number="201" name="201bmp" color="2" fill="10" visible="yes" active="yes"/>
@@
 <part name="SUPPLY16" library="supply2" deviceset="GND" device=""/>
 <part name="D1" library="SparkFun-DiscreteSemi" deviceset="DIODE" device="PTH" value="1N4001"/>
-<part name="IC1" library="national-semiconductor" deviceset="LM2936?*" device="Z" technology="-5.0"/>
 <part name="C2" library="SparkFun-Passives" deviceset="CAP" device="PTH2" value="0.1uF"/>
 <part name="C4" library="SparkFun-Passives" deviceset="CAP" device="PTH2" value="0.1uF"/>
 <part name="FRAME1" library="SparkFun-Aesthetics" deviceset="FRAME-LETTER" device=""/>
-<part name="J7" library="con-jack" deviceset="JACK-PLUG" device="1"/>
+<part name="SUPPLY17" library="supply2" deviceset="GND" device=""/>
+<part name="R3" library="rcl" deviceset="R-US_" device="0204/5" value="330"/>
+<part name="LED2" library="led" deviceset="LED" device="3MM" value="LED13"/>
+<part name="IC1" library="SparkFun-PowerIC" deviceset="V_REG_78XX" device="-TO-220" value="LM2937-5.0"/>
+<part name="J4" library="SparkFun-Connectors" deviceset="POWER_JACK" device="PTH"/>
 </parts>
 <sheets>
@@
 <instance part="SUPPLY16" gate="GND" x="-15.24" y="-66.04"/>
 <instance part="D1" gate="G$1" x="43.18" y="45.72"/>
-<instance part="IC1" gate="G$1" x="78.74" y="43.18"/>
 <instance part="C2" gate="G$1" x="-101.6" y="-27.94"/>
 <instance part="C4" gate="G$1" x="-68.58" y="43.18" rot="R90"/>
 <instance part="FRAME1" gate="G$1" x="-134.62" y="-91.44"/>
 <instance part="FRAME1" gate="G$2" x="12.7" y="-91.44"/>
-<instance part="J7" gate="G$1" x="20.32" y="40.64"/>
+<instance part="SUPPLY17" gate="GND" x="-25.4" y="-76.2"/>
+<instance part="R3" gate="G$1" x="-25.4" y="-66.04" rot="R90"/>
+<instance part="LED2" gate="G$1" x="-25.4" y="-53.34"/>
+<instance part="IC1" gate="G$1" x="78.74" y="45.72"/>
+<instance part="J4" gate="G$1" x="25.4" y="38.1"/>
 </instances>
 <busses>
@@
 </segment>
 <segment>
-<pinref part="IC1" gate="G$1" pin="GND"/>
 <pinref part="SUPPLY2" gate="GND" pin="GND"/>
-<wire x1="78.74" y1="35.56" x2="78.74" y2="27.94" width="0.1524" layer="91"/>
+<wire x1="78.74" y1="38.1" x2="78.74" y2="27.94" width="0.1524" layer="91"/>
 <wire x1="78.74" y1="27.94" x2="78.74" y2="25.4" width="0.1524" layer="91"/>
-<wire x1="27.94" y1="40.64" x2="27.94" y2="27.94" width="0.1524" layer="91"/>
 <wire x1="27.94" y1="27.94" x2="58.42" y2="27.94" width="0.1524" layer="91"/>
 <junction x="78.74" y="27.94"/>
@@
 <wire x1="78.74" y1="27.94" x2="96.52" y2="27.94" width="0.1524" layer="91"/>
 <wire x1="96.52" y1="27.94" x2="96.52" y2="33.02" width="0.1524" layer="91"/>
-<pinref part="J7" gate="G$1" pin="1"/>
-<pinref part="J7" gate="G$1" pin="2"/>
-<wire x1="25.4" y1="38.1" x2="25.4" y2="40.64" width="0.1524" layer="91"/>
-<wire x1="25.4" y1="40.64" x2="27.94" y2="40.64" width="0.1524" layer="91"/>
-<junction x="25.4" y="40.64"/>
+<pinref part="IC1" gate="G$1" pin="GND"/>
+<pinref part="J4" gate="G$1" pin="GNDBREAK"/>
+<wire x1="27.94" y1="43.18" x2="27.94" y2="27.94" width="0.1524" layer="91"/>
+</segment>
+<segment>
+<pinref part="R3" gate="G$1" pin="1"/>
+<pinref part="SUPPLY17" gate="GND" pin="GND"/>
+<wire x1="-25.4" y1="-71.12" x2="-25.4" y2="-73.66" width="0.1524" layer="91"/>
 </segment>
 </net>
@@
 <pinref part="SUPPLY8" gate="+5V" pin="+5V"/>
 <pinref part="C1" gate="G$1" pin="+"/>
-<pinref part="IC1" gate="G$1" pin="VO"/>
 <wire x1="96.52" y1="45.72" x2="96.52" y2="53.34" width="0.1524" layer="91"/>
-<wire x1="88.9" y1="45.72" x2="96.52" y2="45.72" width="0.1524" layer="91"/>
+<wire x1="88.9" y1="45.72" x2="91.44" y2="45.72" width="0.1524" layer="91"/>
 <junction x="96.52" y="45.72"/>
+<pinref part="IC1" gate="G$1" pin="OUT"/>
+<wire x1="91.44" y1="45.72" x2="96.52" y2="45.72" width="0.1524" layer="91"/>
+<wire x1="88.9" y1="45.72" x2="86.36" y2="45.72" width="0.1524" layer="91"/>
 </segment>
 <segment>
@@
 <net name="D13" class="0">
 <segment>
-<wire x1="-30.48" y1="-40.64" x2="-7.62" y2="-40.64" width="0.1524" layer="91"/>
 <pinref part="IC2" gate="1" pin="PB5(SCK/PCINT5)"/>
 <pinref part="J3" gate="G$1" pin="6"/>
 <label x="-20.32" y="-40.64" size="1.778" layer="95"/>
+<wire x1="-30.48" y1="-40.64" x2="-25.4" y2="-40.64" width="0.1524" layer="91"/>
+<pinref part="LED2" gate="G$1" pin="A"/>
+<wire x1="-25.4" y1="-40.64" x2="-7.62" y2="-40.64" width="0.1524" layer="91"/>
+<wire x1="-25.4" y1="-50.8" x2="-25.4" y2="-40.64" width="0.1524" layer="91"/>
+<junction x="-25.4" y="-40.64"/>
 </segment>
 </net>
@@
 <segment>
 <pinref part="D1" gate="G$1" pin="C"/>
-<pinref part="IC1" gate="G$1" pin="VIN"/>
 <wire x1="45.72" y1="45.72" x2="58.42" y2="45.72" width="0.1524" layer="91"/>
 <pinref part="C3" gate="G$1" pin="+"/>
-<wire x1="58.42" y1="45.72" x2="68.58" y2="45.72" width="0.1524" layer="91"/>
+<wire x1="58.42" y1="45.72" x2="71.12" y2="45.72" width="0.1524" layer="91"/>
 <wire x1="58.42" y1="45.72" x2="58.42" y2="40.64" width="0.1524" layer="91"/>
 <junction x="58.42" y="45.72"/>
+<pinref part="IC1" gate="G$1" pin="IN"/>
 </segment>
 </net>
 <net name="N$2" class="1">
 <segment>
-<wire x1="27.94" y1="43.18" x2="27.94" y2="45.72" width="0.1524" layer="91"/>
 <pinref part="D1" gate="G$1" pin="A"/>
 <wire x1="27.94" y1="45.72" x2="40.64" y2="45.72" width="0.1524" layer="91"/>
-<pinref part="J7" gate="G$1" pin="3"/>
-<wire x1="25.4" y1="43.18" x2="27.94" y2="43.18" width="0.1524" layer="91"/>
-</segment>
-</net>
+<pinref part="J4" gate="G$1" pin="PWR"/>
+</segment>
+</net>
+<net name="N$4" class="0">
+<segment>
+<pinref part="LED2" gate="G$1" pin="C"/>
+<pinref part="R3" gate="G$1" pin="2"/>
+<wire x1="-25.4" y1="-58.42" x2="-25.4" y2="-60.96" width="0.1524" layer="91"/>
+</segment>
+</net>
